Commit message: new husky setup

File: husky_description/urdf/husky_macro.urdf.xacro (robot description, xacro)
@@ -85,5 +85,5 @@
     <link name="${prefix}lidar_link"/>
     <joint name="${prefix}lidar_joint" type="fixed">
-      <origin xyz="0.375 0 0.321" rpy="0 0 0" />
+      <origin xyz="0.338 0 0.834" rpy="0 0 0" />
       <parent link="${prefix}base_link" />
       <child link="${prefix}lidar_link" />
