Commit message: Add velodyne plugin (#1)

File: husky_description/urdf/husky.urdf.xacro (robot description, xacro)
@@ -6,4 +6,8 @@
   <xacro:arg name="gazebo_controllers" default="$(find husky_control)/config/control.yaml" />
   <xacro:include filename="$(find husky_description)/urdf/husky_macro.urdf.xacro" />
+  <xacro:include filename="$(find velodyne_description)/urdf/VLP-16.urdf.xacro"/>
+  <xacro:VLP-16 parent="lidar_link" name="velodyne" topic="/points" organize_cloud="false" hz="10" samples="440" gpu="false">
+    <origin xyz="0 0 0" rpy="0 0 0" />
+  </xacro:VLP-16>
   <!-- Load husky description -->
   <xacro:husky prefix="$(arg prefix)" />

Commit message: FIx lidar frame name

File: husky_description/urdf/husky.urdf.xacro (robot description, xacro)
@@ -7,6 +7,6 @@
   <xacro:include filename="$(find husky_description)/urdf/husky_macro.urdf.xacro" />
   <xacro:include filename="$(find velodyne_description)/urdf/VLP-16.urdf.xacro"/>
-  <xacro:VLP-16 parent="lidar_link" name="velodyne" topic="/points" organize_cloud="false" hz="10" lasers="32" samples="2048" min_range="0.3" collision_range="0.3" gpu="true">
-    <origin xyz="0 0 0" rpy="0 0 0" />
+  <xacro:VLP-16 parent="base_link" name="lidar_link" topic="/points" organize_cloud="true" hz="10" lasers="32" samples="2048" min_range="0.3" collision_range="0.3" gpu="true">
+    <origin xyz="0.338 0 0.834" rpy="0 0 0" />
   </xacro:VLP-16>
   <!-- Load husky description -->

File: husky_description/urdf/husky_macro.urdf.xacro (robot description, xacro)
@@ -83,10 +83,4 @@
     <gazebo reference="${prefix}imu_link">
     </gazebo>
-    <link name="${prefix}lidar_link"/>
-    <joint name="${prefix}lidar_joint" type="fixed">
-      <origin xyz="0.338 0 0.834" rpy="0 0 0" />
-      <parent link="${prefix}base_link" />
-      <child link="${prefix}lidar_link" />
-    </joint>
     <!-- Husky wheel macros -->
     <xacro:husky_wheel wheel_prefix="${prefix}front_left">

Commit message: Read lidar offset from env and based on sim load the link

File: husky_description/urdf/husky.urdf.xacro (robot description, xacro)
@@ -6,11 +6,11 @@
   <xacro:arg name="gazebo_controllers" default="$(find husky_control)/config/control.yaml" />
   <xacro:include filename="$(find husky_description)/urdf/husky_macro.urdf.xacro" />
-  <xacro:include filename="$(find velodyne_description)/urdf/VLP-16.urdf.xacro"/>
-  <xacro:VLP-16 parent="base_link" name="lidar_link" topic="/points" organize_cloud="true" hz="10" lasers="32" samples="2048" min_range="0.3" collision_range="0.3" gpu="true">
-    <origin xyz="0.338 0 0.834" rpy="0 0 0" />
-  </xacro:VLP-16>
   <!-- Load husky description -->
   <xacro:husky prefix="$(arg prefix)" />
   <xacro:if value="$(arg is_sim)">
+    <xacro:include filename="$(find velodyne_description)/urdf/VLP-16.urdf.xacro"/>
+    <xacro:VLP-16 parent="base_link" name="lidar_link" topic="/points" organize_cloud="true" hz="10" lasers="32" samples="2048" min_range="0.3" collision_range="0.3" gpu="true">
+      <origin xyz="0.338 0 0.834" rpy="0 0 0" />
+    </xacro:VLP-16>
     <gazebo>
       <plugin name="$(arg prefix)gazebo_ros2_control" filename="libgazebo_ros2_control.so">

File: husky_description/urdf/husky_macro.urdf.xacro (robot description, xacro)
@@ -77,5 +77,5 @@
     <link name="${prefix}imu_link"/>
     <joint name="${prefix}imu_joint" type="fixed">
-      <origin xyz="$(optenv HUSKY_IMU_XYZ 0.19 0 0.149)" rpy="$(optenv HUSKY_IMU_RPY 0 -1.5708 3.1416)" />
+      <origin xyz="$(optenv HUSKY_IMU_XYZ 0.624 0.175 0.040)" rpy="$(optenv HUSKY_IMU_RPY 0 -1.5708 3.1416)" />
       <parent link="${prefix}base_link" />
       <child link="${prefix}imu_link" />
@@ -83,4 +83,12 @@
     <gazebo reference="${prefix}imu_link">
     </gazebo>
+    <xacro:if value="$(arg not is_sim)">
+      <link name="${prefix}lidar_link"/>
+      <joint name="${prefix}lidar_joint" type="fixed">
+        <origin xyz="$(optenv HUSKY_LIDAR_XYZ 0.6055 0 0.285)" rpy="$(optenv HUSKY_LIDAR_RPY 0 0 0)" />
+        <parent link="${prefix}base_link" />
+        <child link="${prefix}lidar_link" />
+      </joint>
+    </xacro>
     <!-- Husky wheel macros -->
     <xacro:husky_wheel wheel_prefix="${prefix}front_left">

Commit message: Fix IMU issue and update velodune gazebo plugin

File: husky_description/urdf/husky.urdf.xacro (robot description, xacro)
@@ -9,6 +9,6 @@
   <xacro:husky prefix="$(arg prefix)" />
   <xacro:if value="$(arg is_sim)">
-    <xacro:include filename="$(find velodyne_description)/urdf/VLP-16.urdf.xacro"/>
-    <xacro:VLP-16 parent="base_link" name="lidar_link" topic="/points" organize_cloud="true" hz="10" lasers="32" samples="2048" min_range="0.3" collision_range="0.3" gpu="true">
+    <xacro:include filename="$(find husky_description)/urdf/accessories/VLP-16.urdf.xacro"/>
+    <xacro:VLP-16 parent="base_link" name="lidar_link" topic="/points" hz="10" lasers="32" gpu="true">
       <origin xyz="0.338 0 0.834" rpy="0 0 0" />
     </xacro:VLP-16>
@@ -18,5 +18,5 @@
       </plugin>
     </gazebo>
-    <gazebo reference="$(arg prefix)base_link">
+    <gazebo reference="$(arg prefix)imu_link">
       <sensor name="imu_sensor" type="imu">
         <always_on>true</always_on>
@@ -70,5 +70,5 @@
             </ros>
             <initial_orientation_as_reference>false</initial_orientation_as_reference>
-            <frame_name>$(arg prefix)base_link</frame_name>
+            <frame_name>$(arg prefix)imu_link</frame_name>
         </plugin>
       </sensor>

File: husky_description/urdf/husky_macro.urdf.xacro (robot description, xacro)
@@ -78,9 +78,7 @@
     <joint name="${prefix}imu_joint" type="fixed">
       <origin xyz="$(optenv HUSKY_IMU_XYZ 0.624 0.175 0.040)" rpy="$(optenv HUSKY_IMU_RPY 0 -1.5708 3.1416)" />
-      <parent link="${prefix}base_link" />
+      <parent link="${prefix}lidar_link" />
       <child link="${prefix}imu_link" />
     </joint>
-    <gazebo reference="${prefix}imu_link">
-    </gazebo>
     <xacro:unless value="$(arg is_sim)">
       <link name="${prefix}lidar_link"/>
